Commit message: 1111 	новый файл:    widowx_arm/test3/.setup_assistant 	новый файл:    widowx_arm/test3/CMakeLists.txt 	новый файл:    widowx_arm/test3/config/cartesian_limits.yaml 	новый файл:    widowx_arm/test3/config/chomp_planning.yaml 	новый файл:    widowx_arm/test3/config/fake_controllers.yaml 	новый файл:    widowx_arm/test3/config/gazebo_controllers.yaml 	новый файл:    widowx_arm/test3/config/joint_limits.yaml 	новый файл:    widowx_arm/test3/config/kinematics.yaml 	новый файл:    widowx_arm/test3/config/ompl_planning.yaml 	новый файл:    widowx_arm/test3/config/ros_controllers.yaml 	новый файл:    widowx_arm/test3/config/sensors_3d.yaml 	новый файл:    widowx_arm/test3/config/simple_moveit_controllers.yaml 	новый файл:    widowx_arm/test3/config/stomp_planning.yaml 	новый файл:    widowx_arm/test3/config/widowx_arm.srdf 	новый файл:    widowx_arm/test3/launch/chomp_planning_pipeline.launch.xml 	новый файл:    widowx_arm/test3/launch/default_warehouse_db.launch 	новый файл:    widowx_arm/test3/launch/demo.launch 	новый файл:    widowx_arm/test3/launch/demo_gazebo.launch 	новый файл:    widowx_arm/test3/launch/fake_moveit_controller_manager.launch.xml 	новый файл:    widowx_arm/test3/launch/gazebo.launch 	новый файл:    widowx_arm/test3/launch/joystick_control.launch 	новый файл:    widowx_arm/test3/launch/move_group.launch 	новый файл:    widowx_arm/test3/launch/moveit.rviz 	новый файл:    widowx_arm/test3/launch/moveit_rviz.launch 	новый файл:    widowx_arm/test3/launch/ompl-chomp_planning_pipeline.launch.xml 	новый файл:    widowx_arm/test3/launch/ompl_planning_pipeline.launch.xml 	новый файл:    widowx_arm/test3/launch/pilz_industrial_motion_planner_planning_pipeline.launch.xml 	новый файл:    widowx_arm/test3/launch/planning_context.launch 	новый файл:    widowx_arm/test3/launch/planning_pipeline.launch.xml 	новый файл:    widowx_arm/test3/launch/ros_control_moveit_controller_manager.launch.xml 	новый файл:    widowx_arm/test3/launch/ros_controllers.launch 	новый файл:    widowx_arm/test3/launch/run_benchmark_ompl.launch 	новый файл:    widowx_arm/test3/launch/sensor_manager.launch.xml 	новый файл:    widowx_arm/test3/launch/setup_assistant.launch 	новый файл:    widowx_arm/test3/launch/simple_moveit_controller_manager.launch.xml 	новый файл:    widowx_arm/test3/launch/stomp_planning_pipeline.launch.xml 	новый файл:    widowx_arm/test3/launch/trajectory_execution.launch.xml 	новый файл:    widowx_arm/test3/launch/warehouse.launch 	новый файл:    widowx_arm/test3/launch/warehouse_settings.launch.xml 	новый файл:    widowx_arm/test3/launch/widowx_arm_moveit.launch 	новый файл:    widowx_arm/test3/launch/widowx_arm_moveit_sensor_manager.launch.xml 	новый файл:    widowx_arm/test3/package.xml 	новый файл:    widowx_arm/test3/scripts/widowx_move.py 	новый файл:    widowx_arm/widowx_arm_description/robots/widowx_arm.urdf 	изменено:      widowx_arm/widowx_arm_description/urdf/widowx.urdf.xacro 	новый файл:    widowx_arm/widowx_arm_description/urdf/widowx.xacro

File: widowx_arm/widowx_arm_description/urdf/widowx.urdf.xacro (robot description, xacro)
@@ -131,5 +131,5 @@
          </inertial>
       </link>
-      <!--link name="${prefix}gripper_rail_link">
+      <link name="${prefix}gripper_rail_link">
          <visual>
             <origin xyz="0 0 0" rpy="0 0 1.57" />
@@ -150,8 +150,8 @@
             <inertia ixx="1.0" ixy="0.0" ixz="0.0" iyy="1.0" iyz="0.0" izz="1.0" />
          </inertial>
-      </link-->
-      <!--link name="${prefix}gripper_aux_link">
-      </link-->
-      <!--link name="${prefix}gripper_1_link">
+      </link>
+      <link name="${prefix}gripper_aux_link">
+      </link>
+      <link name="${prefix}gripper_1_link">
          <visual>
             <origin xyz="0 -0.0007 0" rpy="0 0 1.57" />
@@ -192,5 +192,5 @@
             <inertia ixx="1.0" ixy="0.0" ixz="0.0" iyy="1.0" iyz="0.0" izz="1.0" />
          </inertial>
-      </link-->
+      </link>
       <!-- joints -->
       <joint name="${prefix}arm_base_joint" type="fixed">
@@ -235,5 +235,5 @@
          <limit lower="-2.617" upper="2.617" effort="6" velocity="1.571" />
       </joint>
-      <!--joint name="${prefix}joint_6" type="fixed">
+      <joint name="${prefix}joint_6" type="fixed">
          <origin xyz = "0 0 ${M_SCALE*43}" rpy="0 0 0" />
          <parent link="${prefix}wrist_2_link" />
@@ -241,6 +241,6 @@
          <axis xyz="0 0 1" />
          <limit lower="-0.31" upper="0.1" effort="6" velocity="0.5" />
-      </joint-->
-      <!--joint name="${prefix}gripper_revolute_joint" type="revolute">
+      </joint>
+      <joint name="${prefix}gripper_revolute_joint" type="revolute">
          <origin xyz = "0 0 0.065" rpy="0 0 0" />
          <parent link="${prefix}wrist_2_link" />
@@ -248,6 +248,6 @@
          <axis xyz="0 0 1" />
          <limit lower="-2.6" upper="2.6" effort="6" velocity="0.5" />
-      </joint-->
-      <!--joint name="${prefix}gripper_prismatic_joint_1" type="prismatic">
+      </joint>
+      <joint name="${prefix}gripper_prismatic_joint_1" type="prismatic">
          <origin xyz="0 0 0" rpy="0 0 0" />
          <parent link="${prefix}gripper_rail_link" />
@@ -263,7 +263,6 @@
          <axis xyz="0 1 0" />
          <limit lower="0" upper="0.027" effort="6" velocity="0.5" />
-      </joint-->
+      </joint>
       <!-- gripper -->
-  <xacro:include filename="$(find widowx_arm_description)/urdf/widowx_gripper.xacro"/>
   <!--link name="gripper_link"/>
     <joint name="gripper_link_joint" type="revolute">
