Commit message: trying to setup gripper via editing urdf and py

File: widowx_arm/widowx_arm_description/urdf/widowx_arm.urdf (robot description, URDF)
Before this commit: robot widowx_arm, 7 links, 6 joints
Links:
- added link gripper_1_link, mass 1; collision mesh filename=package://widowx_arm_description/meshes/gripper_hand_fixed_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; visual mesh filename=package://widowx_arm_description/meshes/gripper_hand_fixed_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
- added link gripper_2_link, mass 1; collision mesh filename=package://widowx_arm_description/meshes/gripper_hand_fixed_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; visual mesh filename=package://widowx_arm_description/meshes/gripper_hand_fixed_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
- added link gripper_rail_link, mass 1; collision mesh filename=package://widowx_arm_description/meshes/gripper_rail_link.s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; visual mesh filename=package://widowx_arm_description/meshes/gripper_rail_link.s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
Joints:
- added joint gripper_prismatic_joint_2: type prismatic, parent gripper_rail_link, child gripper_2_link, origin xyz=0 0 0 rpy=0 0 0, axis 0 1 0, limit lower=0.002 upper=0.031 effort=0 velocity=0.5, mimic joint=joint_6
- added joint gripper_rail_joint: type fixed, parent wrist_2_link, child gripper_rail_link, origin xyz=0 0 0.043 rpy=0 0 0, axis 0 0 1
- added joint joint_6: type prismatic, parent gripper_rail_link, child gripper_1_link, origin xyz=0 0 0 rpy=0 0 0, axis 0 -1 0, limit lower=0.002 upper=0.031 effort=0 velocity=0.5
- joint joint_2: limit lower=-1.571 upper=1.571 effort=6 velocity=1.571 -> lower=-3.14 upper=3.14 effort=6 velocity=1.571

Commit message: fixed collision and gripper appearance in rviz

File: widowx_arm/widowx_arm_description/urdf/widowx_arm.urdf (robot description, URDF)
Before this commit: robot widowx_arm, 10 links, 9 joints
Joints:
- joint gripper_prismatic_joint_2: limit lower=0.002 upper=0.031 effort=0 velocity=0.5 -> lower=0.002 upper=0.02 effort=0 velocity=0.5
- joint joint_6: limit lower=0.002 upper=0.031 effort=0 velocity=0.5 -> lower=0.002 upper=0.02 effort=0 velocity=0.5
